Commit message: Reconfigure RViz and Gazebo for visualization and simulation

File: dustbuster_ws/description/robot_draft.urdf (robot description, URDF)
Before this commit: robot robot_draft, 4 links, 3 joints
Links:
- added link laser_frame, mass 0.130033; collision box size=0.050011 0.050011 0.035003; collision cylinder length=0.035003 radius=0.02
Joints:
- added joint laser_joint: type fixed, parent chassis, child laser_frame, origin xyz=0 0.25 0.25 rpy=0 0 1.570796
