Commit message: Reconfigure the env to adapt new plugins, modify the .launch to run also slam

File: dustbuster_ws/description/lidar_2d.xacro (robot description, xacro)
@@ -11,5 +11,5 @@
         <origin xyz="0 0 0" rpy="0 -0 1.5707"/>
         <geometry>
-          <mesh filename="https://fuel.ignitionrobotics.org/1.0/khulqu15/models/lidar 2d v1/1/files/meshes/lidar_2d_v1.dae"/>
+          <mesh filename="file:///home/onur/Desktop/DustBusterAI-Software/dustbuster_ws/description/mesh/lidar_2d_v1.dae"/>
         </geometry>
       </visual>

File: dustbuster_ws/description/robot_draft.urdf (robot description, URDF)
Before this commit: robot robot_draft, 5 links, 4 joints
Links:
- added link base_footprint, mass 0.001
Joints:
- added joint base_footprint_joint: type fixed, parent chassis, child base_footprint, origin xyz=0 0 0 rpy=0 0 0

File: dustbuster_ws/description/robot_draft.urdf.xacro (robot description, xacro)
@@ -2,5 +2,5 @@
 <robot xmlns:xacro="http://www.ros.org/wiki/xacro" name="robot_draft">
   <xacro:include filename="lidar_2d.xacro" />
-  <material name="blackfsdf">
+  <material name="black">
         <color rgba="0 0 0 1" />
     </material>
@@ -16,5 +16,5 @@
         <cylinder radius="0.0601226" length="0.0320289"/>
       </geometry>
-      <material name="blackfsdf"/>
+      <material name="black"/>
     </visual>
     <collision name="collision">
@@ -36,5 +36,5 @@
         <cylinder radius="0.5" length="0.0966706"/>
       </geometry>
-      <material name="blackfsdf"/>
+      <material name="black"/>
     </visual>
     <collision name="collision">
@@ -56,5 +56,5 @@
         <cylinder radius="0.216015" length="0.071441"/>
       </geometry>
-      <material name="blackfsdf"/>
+      <material name="black"/>
     </visual>
     <collision name="collision">
@@ -76,5 +76,5 @@
         <cylinder radius="0.216015" length="0.071441"/>
       </geometry>
-      <material name="blackfsdf"/>
+      <material name="black"/>
     </visual>
     <collision name="collision">
@@ -114,3 +114,6 @@
     <plugin name='wheel_velocity_setter' filename='libwheel_velocity_setter.so'/>
   </gazebo>
+  <gazebo>
+    <plugin name='diff_drive_wheel_encoder' filename='libdiff_drive_wheel_encoder.so'/>
+  </gazebo>
 </robot>
