Commit message: Tune nav2 params for current geometry, modify urdf to arrange center of robot, set rviz config

File: dustbuster_ws/launch/description/dustbuster.urdf (robot description, URDF)
Before this commit: robot robot, 9 links, 8 joints
Joints:
- joint chassis_joint: origin xyz=-0.226 0 -0.01 -> xyz=0 0 0
- joint left_wheel_joint: origin xyz=-0.25 0.58 0 rpy=-1.5707963267948966 0 0 -> xyz=-0.024 0.58 0 rpy=-1.5707963267948966 0 0
- joint right_wheel_joint: origin xyz=-0.25 -0.58 0 rpy=1.5707963267948966 0 0 -> xyz=-0.024 -0.58 0 rpy=1.5707963267948966 0 0

Commit message: Rework URDF for v1 to improve accuracy and realism of the model, set mesh and geometric features

File: dustbuster_ws/launch/description/dustbuster.urdf (robot description, URDF)
Before this commit: robot dustbuster, 9 links, 8 joints
Links:
- link caster_wheel: mass 0.5 -> 0.1; geometry collision cylinder length=0.02 radius=0.035; visual cylinder length=0.02 radius=0.035
- link chassis: mass 20 -> 22.5; geometry collision mesh filename=file:///home/onur/Desktop/DustBusterAI-Software/dustbuster_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; visual mesh filename=file:///home/onur/Desktop/DustBusterAI-Software/dustbuster_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
- link left_wheel: mass 1.5 -> 0.5; geometry collision cylinder length=0.05 radius=0.1225; visual cylinder length=0.05 radius=0.1225
- link right_wheel: mass 1.5 -> 0.5; geometry collision cylinder length=0.05 radius=0.1225; visual cylinder length=0.05 radius=0.1225
Joints:
- joint camera_optical_joint: origin xyz=0 0 0 rpy=-1.5707963267948966 0 -1.5707963267948966 -> xyz=0.5 0 0 rpy=-1.5707963267948966 0 -1.5707963267948966
- joint caster_wheel_joint: origin xyz=0.35 0 -0.15 rpy=1.5707963267948966 0 0 -> xyz=0.35 0 -0.09 rpy=1.5707963267948966 0 0
- joint left_wheel_joint: origin xyz=-0.024 0.58 0 rpy=-1.5707963267948966 0 0 -> xyz=0 0.2935 0 rpy=-1.5707963267948966 0 0
- joint right_wheel_joint: origin xyz=-0.024 -0.58 0 rpy=1.5707963267948966 0 0 -> xyz=0 -0.2935 0 rpy=1.5707963267948966 0 0

Commit message: Rework URDF for v2 to set actual inertial data, caster wheel mount mechanism and nav2 footprint shape of the vehicle

File: dustbuster_ws/launch/description/dustbuster.urdf (robot description, URDF)
Before this commit: robot dustbuster, 9 links, 8 joints
Links:
- added link caster_wheel_mount, mass 0.1; collision box size=0.05 0.05 0.01; visual box size=0.025 0.025 0.06
- link camera_link: mass None -> 3.0
Joints:
- added joint caster_wheel_mount_joint: type revolute, parent chassis, child caster_wheel_mount, origin xyz=0.35 0 -0.065 rpy=0 0 0, axis 0 0 1, limit lower=-3.14159265 upper=3.14159265 effort=1.0 velocity=2.0
- joint caster_wheel_joint: axis (none) -> 0 0 1; limit (none) -> lower=-3.14159265 upper=3.14159265 effort=1.0 velocity=2.0; origin xyz=0.35 0 -0.09 rpy=1.5707963267948966 0 0 -> xyz=0 0 -0.025 rpy=1.5707963267948966 0 0; parent chassis -> caster_wheel_mount; type fixed -> revolute
