Commit message: Integrate IMU and tune Cartographer to get better results, update inertial features of URDF

File: dustbuster_ws/src/dustbuster_launch/dustbuster_launch/description/dustbuster.urdf (robot description, URDF)
Before this commit: robot dustbuster, 10 links, 9 joints
Links:
- added link imu_link, mass 0.01; visual box size=0.01 0.01 0.01
- link camera_link: mass 3.0 -> 3.1
- link caster_wheel_mount: geometry collision box size=0.025 0.025 0.06; visual box size=0.025 0.025 0.06
Joints:
- added joint imu_joint: type fixed, parent base_link, child imu_link, origin xyz=0 0 0 rpy=0 0 0
- joint caster_wheel_joint: limit lower=-3.14159265 upper=3.14159265 effort=1.0 velocity=2.0 -> lower=-100000000000000000000 upper=100000000000000000000 effort=1.0 velocity=2.0
- joint caster_wheel_mount_joint: limit lower=-3.14159265 upper=3.14159265 effort=1.0 velocity=2.0 -> lower=-100000000000000000000 upper=100000000000000000000 effort=1.0 velocity=2.0; origin xyz=0.35 0 -0.065 rpy=0 0 0 -> xyz=0.35 0 -0.0625 rpy=0 0 0

Commit message: Add filter for IMU, optimize localization and mapping, add map for cartographer

File: dustbuster_ws/src/dustbuster_launch/dustbuster_launch/description/dustbuster.urdf (robot description, URDF)
Before this commit: robot dustbuster, 11 links, 10 joints
Links:
- link left_wheel: mass 0.5 -> 0.75; geometry collision cylinder length=0.28 radius=0.1225; visual cylinder length=0.05 radius=0.1225
- link right_wheel: mass 0.5 -> 0.75; geometry collision cylinder length=0.28 radius=0.1225; visual cylinder length=0.05 radius=0.1225
Joints:
- joint left_wheel_joint: origin xyz=0 0.2935 0 rpy=-1.5707963267948966 0 0 -> xyz=0 0.1535 0 rpy=-1.5707963267948966 0 0
- joint right_wheel_joint: origin xyz=0 -0.2935 0 rpy=1.5707963267948966 0 0 -> xyz=0 -0.1535 0 rpy=1.5707963267948966 0 0

Commit message: Improve Cartographer map-to-odom stability by adjusting parameters and sensor configuration

File: dustbuster_ws/src/dustbuster_launch/dustbuster_launch/description/dustbuster.urdf (robot description, URDF)
Before this commit: robot dustbuster, 11 links, 10 joints
Links:
- link left_wheel: mass 0.75 -> 0.5; geometry collision cylinder length=0.05 radius=0.1225; visual cylinder length=0.05 radius=0.1225
- link right_wheel: mass 0.75 -> 0.5; geometry collision cylinder length=0.05 radius=0.1225; visual cylinder length=0.05 radius=0.1225
Joints:
- joint left_wheel_joint: origin xyz=0 0.1535 0 rpy=-1.5707963267948966 0 0 -> xyz=0 0.2935 0 rpy=-1.5707963267948966 0 0
- joint right_wheel_joint: origin xyz=0 -0.1535 0 rpy=1.5707963267948966 0 0 -> xyz=0 -0.2935 0 rpy=1.5707963267948966 0 0
